Commit message: updated robot description and gazebo pkg

File: ros_ws/src/robot_description/urdf/simple.urdf (robot description, URDF)
Before this commit: robot urdfbot, 2 links, 1 joints
Links:
- added link link1, mass 7.20094; collision box size=0.1 0.1 0.1; visual box size=0.1 0.1 0.1
- link base_link: geometry 
- link head_link: mass None -> 7.20094; geometry collision box size=0.1 0.1 0.1; visual box size=0.1 0.1 0.1
Joints:
- added joint joint_base_link_link1: type fixed, parent base_link, child link1, origin xyz=0 0 0 rpy=0 0 0
- joint base_link_to_head_link_joint: origin xyz=0 0 0.12 rpy=0 0 0 -> xyz=0 0 0.11 rpy=0 0 0; parent base_link -> link1
